Commit message: dump

File: src/uirover_description/xacro/drubotara_description.xacro (robot description, xacro)
@@ -102,5 +102,5 @@
   </collision>
 </link>
-<link name="camera_link">
+<link name="zed2i_base_link">
   <inertial>
     <origin xyz="-0.0038644930255475884 -0.00046519988354149487 0.014942744960595" rpy="0 0 0"/>
@@ -122,4 +122,9 @@
   </collision>
 </link>
+<link name="zed2i_camera_center"/>
+<link name="zed2i_left_camera_frame"/>
+<link name="zed2i_left_camera_optical_frame"/>
+<link name="zed2i_right_camera_frame"/>
+<link name="zed2i_right_camera_optical_frame"/>
 <link name="imu_link">
   <inertial>
@@ -227,8 +232,33 @@
   <axis xyz="0 1 0"/>
 </joint>
-<joint name="camera_joint" type="fixed">
+<joint name="zed2i_base_joint" type="fixed">
   <origin xyz="0.4775 -0.001498 0.537" rpy="0 0 0"/>
   <parent link="base_link"/>
-  <child link="camera_link"/>
+  <child link="zed2i_base_link"/>
+</joint>
+<joint name="zed2i_camera_center_joint" type="fixed">
+  <origin xyz="0.0 0.0 0.0" rpy="0 0 0"/>
+  <parent link="zed2i_base_link"/>
+  <child link="zed2i_camera_center"/>
+</joint>
+<joint name="zed2i_left_camera_joint" type="fixed">
+  <origin xyz="0.0 0.06 0.0" rpy="0 0 0"/>
+  <parent link="zed2i_camera_center"/>
+  <child link="zed2i_left_camera_frame"/>
+</joint>
+<joint name="zed2i_left_camera_optical_joint" type="fixed">
+  <origin xyz="0.0 0.0 0.0" rpy="-1.5708 0.0 -1.5708"/>
+  <parent link="zed2i_left_camera_frame"/>
+  <child link="zed2i_left_camera_optical_frame"/>
+</joint>
+<joint name="zed2i_right_camera_joint" type="fixed">
+  <origin xyz="0.0 -0.06 0.0" rpy="0 0 0"/>
+  <parent link="zed2i_camera_center"/>
+  <child link="zed2i_right_camera_frame"/>
+</joint>
+<joint name="zed2i_right_camera_optical_joint" type="fixed">
+  <origin xyz="0.0 0.0 0.0" rpy="-1.5708 0.0 -1.5708"/>
+  <parent link="zed2i_right_camera_frame"/>
+  <child link="zed2i_right_camera_optical_frame"/>
 </joint>
 <joint name="imu_joint" type="fixed">

File: src/uirover_description/xacro/sensors.urdf.xacro (robot description, xacro)
@@ -1,17 +1,17 @@
 <?xml version="1.0"?>
 <robot name="drubotara" xmlns:xacro="http://www.ros.org/wiki/xacro">
-    <gazebo reference="camera_link">
-        <sensor name="camera_sensor" type="depth">
+    <gazebo reference="zed2i_left_camera_frame">
+        <sensor name="zed2i_left_camera_sensor" type="depth">
             <camera>
                 <horizontal_fov>1.91972</horizontal_fov>
                 <vertical_fov>1.22173</vertical_fov>
                 <image>
-                    <width>640</width>
-                    <height>480</height>
+                    <width>1280</width>
+                    <height>720</height>
                     <format>R8G8B8</format>
                 </image>
                 <clip>
                     <near>0.3</near>
-                    <far>10.0</far>
+                    <far>20.0</far>
                 </clip>
             </camera>
@@ -19,27 +19,21 @@
             <update_rate>30</update_rate>
             <visualize>false</visualize>
-            <plugin name="depth_camera_controller" filename="libgazebo_ros_camera.so">
+            <plugin name="zed2i_camera_controller" filename="libgazebo_ros_camera.so">
                 <ros>
-                    <namespace>/</namespace>
-                    <remapping>image_raw:=camera/image_raw</remapping>
-                    <remapping>camera_info:=camera/camera_info</remapping>
-                    <remapping>depth/image_raw:=camera/depth/image_raw_unused</remapping>
-                    <remapping>depth/camera_info:=camera/depth/camera_info_unused</remapping>
-                    <remapping>points:=camera/points</remapping>
+                    <namespace>/zed2i</namespace>
+                    <remapping>image_raw:=left/image_raw</remapping>
+                    <remapping>camera_info:=left/camera_info</remapping>
+                    <remapping>depth/image_raw:=depth/depth_registered</remapping>
+                    <remapping>depth/camera_info:=depth/camera_info</remapping>
+                    <remapping>points:=point_cloud/cloud_registered</remapping>
                 </ros>
-                <camera_name>camera</camera_name>
-                <frame_name>camera_optical_frame</frame_name>
-                <hack_baseline>0.07</hack_baseline>
+                <camera_name>zed2i</camera_name>
+                <frame_name>zed2i_left_camera_optical_frame</frame_name>
+                <hack_baseline>0.12</hack_baseline>
                 <min_depth>0.3</min_depth>
-                <max_depth>10.0</max_depth>
+                <max_depth>20.0</max_depth>
             </plugin>
         </sensor>
     </gazebo>
-    <link name="camera_optical_frame" />
-    <joint name="camera_optical_joint" type="fixed">
-        <origin xyz="0.0 0.0 0.0" rpy="-1.5708 0.0 -1.5708" />
-        <parent link="camera_link" />
-        <child link="camera_optical_frame" />
-    </joint>
     <gazebo reference="imu_link">
         <sensor name="imu_sensor" type="imu">
